File: nixi clock/nixi clock.kicad_sch (KiCad schematic)
At the start: 21 parts, among them IC1 ESP32-S3-WROOM-1U-N4, IC2 74AHCT595PW-Q100,1, IC3 74AHCT595PW-Q100,1, IC4 PCF85063AT_AY, IC5 74141, IC6 74141, IC7 74141, IC8 74141, IC9 LM1117MP-3.3_NOPB, J1 Conn_01x02, J2 Conn_01x02

Commit message: nixi clock
first pcb version
Parts:
- removed J2: Conn_01x02, symbol Connector_Generic:Conn_01x02
- removed N1, N2, N3, N4: ~, nixies-us:nixies-us-IN-4-DSUB, symbol nixies-us:IN-4
- added C10, C11, C4, C6, C7, C8, C9: 10u, Capacitor_SMD:C_0805_2012Metric_Pad1.18x1.45mm_HandSolder, symbol Device:C
- added C5: TMCP0G476MTR2F, CAPPM2012X120N, symbol SamacSys_Parts:TMCP0G476MTR2F
- added H1, H2, H3, H4: MountingHole_Pad, MountingHole:MountingHole_3.2mm_M3_Pad_Via, symbol Mechanical:MountingHole_Pad
- added J2, J7: Conn_01x01, Connector_PinHeader_2.54mm:PinHeader_1x01_P2.54mm_Vertical, symbol Connector_Generic:Conn_01x01
- added J3, J4: Conn_01x04, Connector_PinHeader_2.54mm:PinHeader_1x04_P2.54mm_Vertical, symbol Connector_Generic:Conn_01x04
- added J5, J6: Conn_01x02, Connector_PinHeader_2.54mm:PinHeader_1x02_P2.54mm_Vertical, symbol Connector_Generic:Conn_01x02
- added R1, R2: 4k7, Resistor_SMD:R_0805_2012Metric_Pad1.20x1.40mm_HandSolder, symbol Device:R
- added R7: 10k, Resistor_SMD:R_0805_2012Metric_Pad1.20x1.40mm_HandSolder, symbol Device:R
- C1, C2, C3: value C -> 10u; footprint Capacitor_SMD:C_0805_2012Metric -> Capacitor_SMD:C_0805_2012Metric_Pad1.18x1.45mm_HandSolder
- J1: footprint (none) -> Connector_PinHeader_2.54mm:PinHeader_1x02_P2.54mm_Vertical
Connections:
- net +3.3V: now also C5.1 (+), J4.4 (Pin_4), R7.1
- net +5V: now also C10.2, C11.2, C6.2, C7.2, C8.2, C9.2, J3.1 (Pin_1), R1.1, R2.1
- net D_CLK: now also IC1.10 (IO17); no longer IC1.31 (IO38)
- net GND: now also C10.1, C11.1, C4.2, C5.2 (-), C6.1, C7.1, C8.1, C9.1, H1.1, H2.1, H3.1, H4.1, J3.4 (Pin_4), J4.1 (Pin_1), J5.2 (Pin_2), J6.2 (Pin_2), J7.1 (Pin_1)
- net N1A: now also IC5.3
- net N1C: now also IC5.7; no longer IC5.4
- net N1D: now also IC5.4
- net NIXI_DATA: now also IC1.13 (IO19); no longer IC1.28 (IO35)
- net NIXI_EN: now also IC1.12 (IO8); no longer IC1.29 (IO36)
- net O_CLK: now also IC1.11 (IO18); no longer IC1.30 (IO37)
- net RST: now also IC1.9 (IO16)
- net VBUS: now also J2.1 (Pin_1)
- net BOOT: now reaches IC1.27 (IO0)
- net BOOT: now also J6.1 (Pin_1)
- net EN: now reaches IC1.3 (EN)
- net EN: now also C4.1, J5.1 (Pin_1), R7.2
- net RXD: now reaches IC1.36 (RXD0)
- net RXD: now also J4.2 (Pin_2)
- net TXD: now reaches IC1.37 (TXD0)
- net TXD: now also J4.3 (Pin_3)
- new net: J3.3 (Pin_3), R2.2
- new net: J3.2 (Pin_2), R1.2
Other:
- added sheet nixies (nixies.kicad_sch)
